Commit message: change new model

File: src/ec_description/urdf/encos130.xacro (robot description, xacro)
@@ -573,4 +573,33 @@
     <limit lower="-0.6108652" upper="2.0943951" effort="30" velocity="36.34" />
   </joint>
+  <link name="left_wrist_roll_link">
+    <inertial>
+      <origin xyz="0.07979044 0.00049128 0.00044533" rpy="0 0 0" />
+      <mass value="0.99326787" />
+      <inertia ixx="0.00046196" ixy="0.00021671" ixz="-0.00006169" iyy="0.00684056" iyz="0.00000717" izz="0.00679938" />
+    </inertial>
+    <visual>
+      <origin xyz="0 0 0" rpy="0 0 0" />
+      <geometry>
+        <mesh filename="package://ec_description/meshes/left_wrist_roll_link_hand.STL" />
+      </geometry>
+      <material name="">
+        <color rgba="1 1 1 1" />
+      </material>
+    </visual>
+    <collision>
+      <origin xyz="0 0 0" rpy="0 0 0" />
+      <geometry>
+        <mesh filename="package://ec_description/meshes/left_wrist_roll_link_hand.STL" />
+      </geometry>
+    </collision>
+  </link>
+  <joint name="left_wrist_roll_joint" type="revolute">
+    <origin xyz="0.0492 -0.0001 0" rpy="0 0 0" />
+    <parent link="left_elbow_link" />
+    <child link="left_wrist_roll_link" />
+    <axis xyz="1 0 0" />
+    <limit lower="-2.7925268" upper="2.7925268" effort="30" velocity="36.34" />
+  </joint>
   <!-- ==================== Right Arm ==================== -->
   <link name="right_shoulder_pitch_link">
@@ -690,4 +719,33 @@
     <limit lower="-0.6108652" upper="2.0943951" effort="30" velocity="36.34" />
   </joint>
+  <link name="right_wrist_roll_link">
+    <inertial>
+      <origin xyz="0.07979044 -0.00049128 0.00044533" rpy="0 0 0" />
+      <mass value="0.99326787" />
+      <inertia ixx="0.00046196" ixy="-0.00021671" ixz="-0.00006169" iyy="0.00684056" iyz="-0.00000717" izz="0.00679938" />
+    </inertial>
+    <visual>
+      <origin xyz="0 0 0" rpy="0 0 0" />
+      <geometry>
+        <mesh filename="package://ec_description/meshes/right_wrist_roll_link_hand.STL" />
+      </geometry>
+      <material name="">
+        <color rgba="1 1 1 1" />
+      </material>
+    </visual>
+    <collision>
+      <origin xyz="0 0 0" rpy="0 0 0" />
+      <geometry>
+        <mesh filename="package://ec_description/meshes/right_wrist_roll_link_hand.STL" />
+      </geometry>
+    </collision>
+  </link>
+  <joint name="right_wrist_roll_joint" type="revolute">
+    <origin xyz="0.0492 0.0001 0" rpy="0 0 0" />
+    <parent link="right_elbow_link" />
+    <child link="right_wrist_roll_link" />
+    <axis xyz="1 0 0" />
+    <limit lower="-2.7925268" upper="2.7925268" effort="30" velocity="36.34" />
+  </joint>
   <!-- ==================== ros2_control ==================== -->
   <xacro:include filename="$(find ec_description)/urdf/ros2_control.xacro"/>

File: src/ec_description/urdf/ros2_control.xacro (robot description, xacro)
@@ -7,4 +7,5 @@
         <plugin>ec_joint_hardware/EcJointHardware</plugin>
         <param name="config_file">$(find ec_joint_hardware)/config/control.json</param>
+        <param name="log_path">/home/milkyway/log/hunter130</param>
         <param name="adapter_type_0">Ethercat</param>
         <param name="interface_name_0">enp86s0</param>
@@ -223,4 +224,15 @@
         <state_interface name="effort"/>
       </joint>
+      <joint name="${prefix}left_wrist_roll_joint">
+        <command_interface name="position"/>
+        <command_interface name="velocity"/>
+        <command_interface name="effort"/>
+        <command_interface name="kp"/>
+        <command_interface name="kd"/>
+        <command_interface name="torque_mode"/>
+        <state_interface name="position"/>
+        <state_interface name="velocity"/>
+        <state_interface name="effort"/>
+      </joint>
       <!-- Right Arm Joints -->
       <joint name="${prefix}right_shoulder_pitch_joint">
@@ -258,4 +270,15 @@
       </joint>
       <joint name="${prefix}right_elbow_joint">
+        <command_interface name="position"/>
+        <command_interface name="velocity"/>
+        <command_interface name="effort"/>
+        <command_interface name="kp"/>
+        <command_interface name="kd"/>
+        <command_interface name="torque_mode"/>
+        <state_interface name="position"/>
+        <state_interface name="velocity"/>
+        <state_interface name="effort"/>
+      </joint>
+      <joint name="${prefix}right_wrist_roll_joint">
         <command_interface name="position"/>
         <command_interface name="velocity"/>
