Commit message: 修改名字

File: src/ec_description/urdf/ros2_control.xacro (robot description, xacro)
@@ -1,5 +1,5 @@
 <?xml version="1.0"?>
-<robot xmlns:xacro="http://www.ros.org/wiki/xacro" name="encos130_ros2_control">
-  <xacro:macro name="encos130_ros2_control" params="name prefix">
+<robot xmlns:xacro="http://www.ros.org/wiki/xacro" name="hunter130_ros2_control">
+  <xacro:macro name="hunter130_ros2_control" params="name prefix">
     <ros2_control name="${name}" type="system">
       <!-- Joint hardware -->
