Commit message: rename robot to hunter130

File: src/ec_description/urdf/hunter130.xacro (robot description, xacro)
@@ -1,4 +1,4 @@
 <?xml version="1.0" encoding="utf-8"?>
-<robot name="encos130" xmlns:xacro="http://www.ros.org/wiki/xacro">
+<robot name="hunter130" xmlns:xacro="http://www.ros.org/wiki/xacro">
   <!-- ==================== Pelvis (Base) ==================== -->
   <link name="pelvis">
@@ -750,4 +750,4 @@
   <!-- ==================== ros2_control ==================== -->
   <xacro:include filename="$(find ec_description)/urdf/ros2_control.xacro"/>
-  <xacro:encos130_ros2_control name="encos130" prefix=""/>
+  <xacro:hunter130_ros2_control name="hunter130" prefix=""/>
 </robot>

File: src/ec_description/urdf/ros2_control.xacro (robot description, xacro)
@@ -1,5 +1,5 @@
 <?xml version="1.0"?>
-<robot xmlns:xacro="http://www.ros.org/wiki/xacro" name="encos130_ros2_control">
-  <xacro:macro name="encos130_ros2_control" params="name prefix">
+<robot xmlns:xacro="http://www.ros.org/wiki/xacro" name="hunter130_ros2_control">
+  <xacro:macro name="hunter130_ros2_control" params="name prefix">
     <ros2_control name="${name}" type="system">
       <!-- Joint hardware -->
